Commit message: Use meshes for base, head and eyes Revise joint values

File: urdf/mira_simple.urdf (robot description, URDF)
Before this commit: robot mira, 7 links, 6 joints
Links:
- link base_link: geometry visual mesh filename=package://my_mira_description/models/mira/meshes/mira_body_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
- link head_link: geometry visual mesh filename=package://my_mira_description/models/mira/meshes/mira_head_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
- link left_eye_link: geometry visual mesh filename=package://my_mira_description/models/mira/meshes/mira_eye_v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
- link right_eye_link: geometry visual mesh filename=package://my_mira_description/models/mira/meshes/mira_eye_v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
Joints:
- joint base_head_joint: origin xyz=0 0 0 rpy=0 0 0 -> xyz=0 0 0 rpy=0 0 1.57
- joint head_lefteye_joint: origin xyz=0.06 0.01 0 rpy=0 0 0 -> xyz=-0.01 0.06 0.008 rpy=1.57 0 0
- joint head_righteye_joint: origin xyz=0.06 -0.01 0 rpy=0 0 0 -> xyz=0.01 0.06 0.008 rpy=1.57 0 0
- joint roll_joint: origin xyz=0 0 0.08 rpy=0 0 0 -> xyz=0 0 0.03 rpy=0 0 0
