Commit message: Complete mira for gazebo except camera

File: urdf/mira_simple_collisions_inertias2.urdf (robot description, URDF)
Before this commit: robot mira, 2 links, 1 joints
Links:
- added link head_link, mass 0.02; visual mesh filename=package://my_mira_description/models/mira/meshes/mira_head_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
- added link left_eye_link; visual mesh filename=package://my_mira_description/models/mira/meshes/mira_eye_v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
- added link pitch_M2_link, mass 0.001; visual cylinder length=0.005 radius=0.01
- added link right_eye_link; visual mesh filename=package://my_mira_description/models/mira/meshes/mira_eye_v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
- added link roll_M1_link, mass 0.001; visual cylinder length=0.005 radius=0.01
- added link yaw_M3_link, mass 0.001; visual cylinder length=0.005 radius=0.01
Joints:
- added joint base_head_joint: type fixed, parent yaw_M3_link, child head_link, origin xyz=0 0 0 rpy=0 0 1.57
- added joint head_lefteye_joint: type fixed, parent head_link, child left_eye_link, origin xyz=-0.01 0.06 0.008 rpy=1.57 0 0
- added joint head_righteye_joint: type fixed, parent head_link, child right_eye_link, origin xyz=0.01 0.06 0.008 rpy=1.57 0 0
- added joint pitch_joint: type revolute, parent roll_M1_link, child pitch_M2_link, origin xyz=0 0 0 rpy=0 0 0, axis 0 1 0, limit lower=-0.2 upper=0.2 effort=0.1 velocity=0.005
- added joint roll_joint: type revolute, parent body_link, child roll_M1_link, origin xyz=0 0 0.03 rpy=0 0 0, axis 1 0 0, limit lower=-0.2 upper=0.2 effort=0.1 velocity=0.005
- added joint yaw_joint: type revolute, parent pitch_M2_link, child yaw_M3_link, origin xyz=0 0 0 rpy=0 0 0, axis 0 0 1, limit lower=-0.2 upper=0.2 effort=0.1 velocity=0.005

Commit message: Urdf with controllers Only roll joint currently spawns

File: urdf/mira_simple_collisions_inertias2.urdf (robot description, URDF)
Before this commit: robot mira, 8 links, 7 joints
Links:
- link head_link: geometry collision sphere radius=0.06; visual mesh filename=package://my_mira_description/models/mira/meshes/mira_head_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
